File: flexbee.kicad_pcb (KiCad board)
At the start: 4 copper layers, 31 x 17.6 mm, 86 parts, among them J1 Conn_01x12_Male, J2 Conn_01x12_Male, U1 SSD210, U2 ea3056, U3 spinor, Y1 Crystal_GND24

Commit message: Add a photo
Other:
- board text added: "perdita rev1"
- board text removed: "predita rev0"
Changed lines of the file:
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@@
     (effects (font (size 0.8 0.8) (thickness 0.2)) (justify mirror))
   )
-  (gr_text "predita rev0" (at 133.175 97.55) (layer "B.SilkS")
+  (gr_text "perdita rev1" (at 133.175 97.55) (layer "B.SilkS")
     (effects (font (size 0.8 0.8) (thickness 0.2)) (justify mirror))
   )
