File: flexbee.kicad_sch (KiCad schematic)
At the start: 68 parts, among them U1 SSD210, U2 ea3056

Commit message: Get rid of some junk..
Parts:
- C1, C10, C11, C12, C13, C14, C15, C16, C17, C18, C19, C2, C20, C21, C22, C23, C3, C4, C5, C6, C7, C8, C9: value (none) -> C; footprint (none) -> Capacitor_SMD:C_0402_1005Metric
- J1, J2: value (none) -> Conn_01x12_Male; footprint (none) -> Connector_PinHeader_2.54mm:PinHeader_1x12_P2.54mm_Vertical
- L1, L2, L3: value (none) -> L; footprint (none) -> Inductor_SMD:L_Taiyo-Yuden_MD-2020
- R1, R13, R14, R15, R16, R17, R2, R3, R4, R5, R6, R7, R8: value (none) -> R; footprint (none) -> Resistor_SMD:R_0402_1005Metric
- R10, R11, R12, R9: value (none) -> R; footprint (none) -> Capacitor_SMD:C_0402_1005Metric
- TP1, TP5: value (none) -> TestPoint; footprint (none) -> TestPoint:TestPoint_Pad_D1.0mm
- TP6, TP7, TP8: footprint (none) -> TestPoint:TestPoint_Pad_D1.0mm
- U1: footprint (none) -> qfn68_35mm:QFN-68_EP_7x7_Pitch0.35mm
- U2: footprint (none) -> Package_DFN_QFN:QFN-24-1EP_4x4mm_P0.5mm_EP2.7x2.7mm_ThermalVias
- U3: value (none) -> spinor; footprint (none) -> wson8-8x6mm:wson8-8x6mm
- Y1: value (none) -> Crystal_GND24; footprint (none) -> Crystal:Crystal_SMD_Abracon_ABM8G-4Pin_3.2x2.5mm

Commit message: Layout work.
Connections:
- net sar_gpio0: now also J1.5 (Pin_5); no longer J1.3 (Pin_3)
- net sar_gpio2: now also J1.3 (Pin_3); no longer J1.5 (Pin_5)
Changed lines of the file:
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@@
     (effects (font (size 1.27 1.27)) (justify left bottom))
   )
-  (label "sar_gpio2" (at 217.17 186.69 0)
+  (label "sar_gpio2" (at 217.17 181.61 0)
     (effects (font (size 1.27 1.27)) (justify left bottom))
   )
@@
     (effects (font (size 1.27 1.27)) (justify left bottom))
   )
-  (label "sar_gpio0" (at 217.17 181.61 0)
+  (label "sar_gpio0" (at 217.17 186.69 0)
     (effects (font (size 1.27 1.27)) (justify left bottom))
   )
