File: flexbee.kicad_sch (KiCad schematic)
At the start: 68 parts, among them J1 Conn_01x12_Male, J2 Conn_01x12_Male, U1 SSD210, U2 ea3056, U3 spinor, Y1 Crystal_GND24

Commit message: test
Other:
- moved on the sheet: R9
Changed lines of the file:
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@@
     (stroke (width 0) (type default) (color 0 0 0 0))
   )
-  (wire (pts (xy 187.96 49.53) (xy 187.96 62.23))
+  (wire (pts (xy 200.025 50.165) (xy 187.96 62.23))
     (stroke (width 0) (type default) (color 0 0 0 0))
   )
@@
     (stroke (width 0) (type default) (color 0 0 0 0))
   )
-  (wire (pts (xy 187.96 39.37) (xy 187.96 41.91))
+  (wire (pts (xy 187.96 39.37) (xy 200.025 42.545))
     (stroke (width 0) (type default) (color 0 0 0 0))
   )
@@
     (pin "1")
   )
-  (symbol (lib_id "Device:R") (at 187.96 45.72 0) (unit 1)
-    (in_bom yes) (on_board yes) (fields_autoplaced)
-    (property "Reference" "R9" (id 0) (at 190.5 44.4499 0)
-      (effects (font (size 1.27 1.27)) (justify left))
-    )
-    (property "Value" "R" (id 1) (at 190.5 46.9899 0)
-      (effects (font (size 1.27 1.27)) (justify left))
-    )
-    (property "Footprint" "Capacitor_SMD:C_0402_1005Metric" (id 2) (at 186.182 45.72 90)
-      (effects (font (size 1.27 1.27)) hide)
-    )
-    (property "Datasheet" "~" (id 3) (at 187.96 45.72 0)
-      (effects (font (size 1.27 1.27)) hide)
-    )
+  (symbol (lib_id "Device:R") (at 200.025 46.355 0) (unit 1)
+    (in_bom yes) (on_board yes) (fields_autoplaced)
+    (property "Reference" "R9" (id 0) (at 202.565 45.0849 0)
+      (effects (font (size 1.27 1.27)) (justify left))
+    )
+    (property "Value" "R" (id 1) (at 202.565 47.6249 0)
+      (effects (font (size 1.27 1.27)) (justify left))
+    )
+    (property "Footprint" "Capacitor_SMD:C_0402_1005Metric" (id 2) (at 198.247 46.355 90)
+      (effects (font (size 1.27 1.27)) hide)
+    )
+    (property "Datasheet" "~" (id 3) (at 200.025 46.355 0)
+      (effects (font (size 1.27 1.27)) hide)
+    )
